File: HW2/HW2_1/HW2_1.brd (EAGLE design)
At the start: 50 x 50 mm, 22 parts, among them J1 USB-MB-H

Commit message: HW3
Parts:
- moved R2 79.6 mm to (36.8, 10.2), turned to 90 degrees
- moved LED2 77.2 mm to (32.9, 3.43)
- moved C2 76.2 mm to (16.7, 11.1)
- moved J1 75.3 mm to (6.13, 45.4), turned to 270 degrees
- moved U$2 72.6 mm to (18.5, 45.2), flipped to the bottom
- moved U$7 71.5 mm to (1.27, 16.5), turned to 90 degrees
- moved U$4 60.2 mm to (6.92, 4.78), turned to 90 degrees
- moved LED1 57.5 mm to (40.8, 3.04)
- moved C3 54.3 mm to (40.6, 38.8)
- moved R1 54.3 mm to (44.4, 10.6), turned to 90 degrees
- moved R3 45.7 mm to (8.75, 17.5)
- moved R4 41.4 mm to (9.00, 12.8)
- moved C4 39.1 mm to (40.7, 32.3)
- moved U$9 37.1 mm to (15.2, 17.8), turned to 270 degrees
- moved U$8 36.3 mm to (48.9, 46.8), flipped to the top, turned to 270 degrees
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Routing:
- net +3V3: track 0.00 -> 151.1 mm
- net +5V: track 0.00 -> 89.8 mm
- net MCLR: track 0.00 -> 84.4 mm
- net USBID: track 0.00 -> 59.5 mm, vias 0 -> 1
- net B4/USER: track 0.00 -> 47.4 mm
- net A4/LED: track 0.00 -> 43.7 mm
- net D+: track 0.00 -> 41.6 mm
- net PGD: track 0.00 -> 37.9 mm, vias 0 -> 1
- net D-: track 0.00 -> 37.7 mm
- net PGC: track 0.00 -> 36.9 mm
- net B9: track 0.00 -> 24.9 mm
- net B8: track 0.00 -> 24.9 mm
- net B7: track 0.00 -> 24.9 mm
- net A0: track 0.00 -> 22.7 mm
- net A1: track 0.00 -> 22.0 mm
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- added copper zone on layer 16, net GND
Other:
- board text added: "+"
- board text added: "+3V3"
- board text added: "+5V"
- board text added: "A0"
- board text added: "A1"
- board text added: "B13"
- board text added: "B14"
- board text added: "B15"
- board text added: "B2"
- board text added: "B3"
- board text added: "B7"
- board text added: "B8"
- board text added: "B9"
- board text added: "GND"
- board text added: "LED"
- board text added: "MCLR"
- board text added: "PGC"
- board text added: "PGD"
- board text added: "USER"
- board text added: "WILLX"
